File: GPA PCB files/GPA_dortmund_2.sch (KiCad schematic (older format))
At the start: 29 parts, among them U100 AAVID_TO220_HEATSINK, U11 OPA549_KV_11TO-220_11, U12 OPA549_KV_11TO-220_11, U13 INA149SOIC8, X5 MINI-FIT-JR-045569-NA2

Commit message: fixed schematic after conversion from eagle
Parts:
- U11, U12: value OPA549_KV_11TO-220_11 -> OPA549
Connections:
- no-connect marks 0 -> 1
Changed lines of the file:
@@
 $Descr A4 11693 8268
 encoding utf-8
-Sheet 1 6
+Sheet 3 6
 Title ""
 Date ""
@@
 Wire Wire Line
 	4600 2800 5000 2800
-Text GLabel 4700 2800 2    70   BiDi ~ 0
+Text GLabel 5000 2800 2    70   BiDi ~ 0
 VCC
 Wire Wire Line
@@
 Wire Wire Line
 	8000 3000 8400 3000
-Text GLabel 8100 3000 2    70   BiDi ~ 0
+Text GLabel 8400 3000 2    70   BiDi ~ 0
 VCC
 Wire Wire Line
 	9400 4100 9600 4100
-Text GLabel 9400 4100 2    70   BiDi ~ 0
+Text GLabel 9600 4100 2    70   BiDi ~ 0
 VCC
 Wire Wire Line
@@
 Connection ~ 4800 1300
 Connection ~ 5200 1300
-Text GLabel 4200 1300 2    70   BiDi ~ 0
+Text GLabel 4200 1300 0    70   BiDi ~ 0
 VCC
 Wire Wire Line
@@
 Connection ~ 7600 1300
 Connection ~ 8000 1300
-Text GLabel 7000 1300 2    70   BiDi ~ 0
+Text GLabel 7000 1300 0    70   BiDi ~ 0
 VCC
 Wire Wire Line
@@
 	5000 4300 5000 4700
 Connection ~ 5000 4700
-Text GLabel 5300 4700 2    70   BiDi ~ 0
-GND
 Wire Wire Line
 	8000 4500 8000 4700
@@
 	8700 4700 8000 4700
 Connection ~ 7600 4700
-Text GLabel 7200 4700 2    70   BiDi ~ 0
-GND
 Connection ~ 8000 4700
 Wire Wire Line
@@
 Connection ~ 4800 1800
 Connection ~ 4400 1800
-Text GLabel 4200 1800 2    70   BiDi ~ 0
-GND
 Wire Wire Line
 	7000 1800 7200 1800
@@
 Connection ~ 7600 1800
 Connection ~ 7200 1800
-Text GLabel 7000 1800 2    70   BiDi ~ 0
-GND
 Wire Wire Line
 	7100 6000 7200 6000
 Wire Wire Line
 	7200 6000 8300 6000
-Text GLabel 8000 6000 2    70   BiDi ~ 0
-GND
 Connection ~ 7200 6000
 Wire Wire Line
@@
 Wire Wire Line
 	2300 4000 1800 4000
-Text GLabel 1800 4000 2    70   BiDi ~ 0
+Text GLabel 1800 4000 0    70   BiDi ~ 0
 REF_2.5V
 Wire Wire Line
@@
 	5600 6800 4800 6800
 Connection ~ 5600 6800
-Text GLabel 4800 6800 2    70   BiDi ~ 0
+Text GLabel 4800 6800 0    70   BiDi ~ 0
 REF_2.5V
 Wire Wire Line
@@
 Wire Wire Line
 	7200 5700 6900 5700
-Text GLabel 6400 5700 2    70   BiDi ~ 0
+Text GLabel 6400 5700 0    70   BiDi ~ 0
 12V
 Connection ~ 6900 5700
 Wire Wire Line
 	7800 3200 7100 3200
-Text GLabel 7100 3200 2    70   BiDi ~ 0
+Text GLabel 7100 3200 0    70   BiDi ~ 0
 FAULT_OUT_0_1
 Wire Wire Line
 	4800 3200 5400 3200
-Text GLabel 4800 3200 2    70   BiDi ~ 0
+Text GLabel 5400 3200 2    70   BiDi ~ 0
 FAULT_OUT_0_0
 Wire Wire Line
@@
 Wire Wire Line
 	2300 3600 1800 3600
-Text GLabel 1800 3600 2    70   BiDi ~ 0
+Text GLabel 1800 3600 0    70   BiDi ~ 0
 DAC_OUT_3
 Wire Wire Line
 	7600 6700 8300 6700
-Text GLabel 7600 6700 2    70   BiDi ~ 0
+Text GLabel 8300 6700 2    70   BiDi ~ 0
 V_CURRENT_3
 $Comp
@@
 AR Path="/6BED38E3" Ref="U11"  Part="1"
 AR Path="/61AB9CEF/6BED38E3" Ref="U11"  Part="1"
-F 0 "U11" H 5014 4059 69  0000 L BNN
-F 1 "OPA549_KV_11TO-220_11" H 4989 3959 69  0000 L BNN
+F 0 "U11" H 4550 3850 69  0000 L BNN
+F 1 "OPA549" H 4550 3750 69  0000 L BNN
 F 2 "GPA_dortmund:TA11B" H 4700 3800 50  0001 C CNN
 F 3 "" H 4700 3800 50  0001 C CNN
@@
 AR Path="/6D2AEAA6" Ref="U12"  Part="1"
 AR Path="/61AB9CEF/6D2AEAA6" Ref="U12"  Part="1"
-F 0 "U12" H 8814 4059 69  0000 L BNN
-F 1 "OPA549_KV_11TO-220_11" H 7589 3959 69  0000 L BNN
+F 0 "U12" H 7900 3800 69  0000 L BNN
+F 1 "OPA549" H 7700 3700 69  0000 L BNN
 F 2 "GPA_dortmund:TA11B" H 7900 3800 50  0001 C CNN
 F 3 "" H 7900 3800 50  0001 C CNN
@@
 	1    0    0    -1
 $EndComp
+$Comp
+L power:GND #PWR?
+U 1 1 61BC4EC3
+P 8300 6000
+AR Path="/61AB9A1E/61BC4EC3" Ref="#PWR?"  Part="1"
+AR Path="/61AB9CEF/61BC4EC3" Ref="#PWR0123"  Part="1"
+F 0 "#PWR0123" H 8300 5750 50  0001 C CNN
+F 1 "GND" H 8305 5827 50  0000 C CNN
+F 2 "" H 8300 6000 50  0001 C CNN
+F 3 "" H 8300 6000 50  0001 C CNN
+	1    8300 6000
+	1    0    0    -1
+$EndComp
+$Comp
+L power:GND #PWR?
+U 1 1 61BCE2B2
+P 7100 4700
+AR Path="/61AB9A1E/61BCE2B2" Ref="#PWR?"  Part="1"
+AR Path="/61AB9CEF/61BCE2B2" Ref="#PWR0124"  Part="1"
+F 0 "#PWR0124" H 7100 4450 50  0001 C CNN
+F 1 "GND" H 7105 4527 50  0000 C CNN
+F 2 "" H 7100 4700 50  0001 C CNN
+F 3 "" H 7100 4700 50  0001 C CNN
+	1    7100 4700
+	1    0    0    -1
+$EndComp
+$Comp
+L power:GND #PWR?
+U 1 1 61BD761A
+P 5600 4700
+AR Path="/61AB9A1E/61BD761A" Ref="#PWR?"  Part="1"
+AR Path="/61AB9CEF/61BD761A" Ref="#PWR0125"  Part="1"
+F 0 "#PWR0125" H 5600 4450 50  0001 C CNN
+F 1 "GND" H 5605 4527 50  0000 C CNN
+F 2 "" H 5600 4700 50  0001 C CNN
+F 3 "" H 5600 4700 50  0001 C CNN
+	1    5600 4700
+	1    0    0    -1
+$EndComp
+$Comp
+L power:GND #PWR?
+U 1 1 61BE098E
+P 4200 1800
+AR Path="/61AB9A1E/61BE098E" Ref="#PWR?"  Part="1"
+AR Path="/61AB9CEF/61BE098E" Ref="#PWR0126"  Part="1"
+F 0 "#PWR0126" H 4200 1550 50  0001 C CNN
+F 1 "GND" H 4205 1627 50  0000 C CNN
+F 2 "" H 4200 1800 50  0001 C CNN
+F 3 "" H 4200 1800 50  0001 C CNN
+	1    4200 1800
+	1    0    0    -1
+$EndComp
+$Comp
+L power:GND #PWR?
+U 1 1 61BE9C7D
+P 7000 1800
+AR Path="/61AB9A1E/61BE9C7D" Ref="#PWR?"  Part="1"
+AR Path="/61AB9CEF/61BE9C7D" Ref="#PWR0127"  Part="1"
+F 0 "#PWR0127" H 7000 1550 50  0001 C CNN
+F 1 "GND" H 7005 1627 50  0000 C CNN
+F 2 "" H 7000 1800 50  0001 C CNN
+F 3 "" H 7000 1800 50  0001 C CNN
+	1    7000 1800
+	1    0    0    -1
+$EndComp
+NoConn ~ 6600 4300
 $EndSCHEMATC

Commit message: more schematic fixes, only 1 ERC warning left (but thats ok)
Parts:
- U11, U12: symbol GPA_dortmund-eagle-import:OPA549_KV_11TO-220_11 -> GPA_dortmund-rescue:OPA549_KV_11TO-220_11-GPA_dortmund-eagle-import
Connections:
- net labels added: +12V
- net labels removed: 12V
Changed lines of the file:
@@
 Text GLabel 5000 2800 2    70   BiDi ~ 0
 VCC
-Wire Wire Line
-	8000 3100 8000 3000
-Wire Wire Line
-	8000 3000 8400 3000
-Text GLabel 8400 3000 2    70   BiDi ~ 0
+Text GLabel 8200 3000 2    70   BiDi ~ 0
 VCC
 Wire Wire Line
@@
 	7100 6000 7200 6000
 Wire Wire Line
-	7200 6000 8300 6000
+	7200 6000 8000 6000
 Connection ~ 7200 6000
 Wire Wire Line
@@
 Wire Wire Line
 	7200 5700 6900 5700
-Text GLabel 6400 5700 0    70   BiDi ~ 0
-12V
 Connection ~ 6900 5700
 Wire Wire Line
-	7800 3200 7100 3200
-Text GLabel 7100 3200 0    70   BiDi ~ 0
+	7800 3200 7700 3200
+Text GLabel 7700 3200 0    70   BiDi ~ 0
 FAULT_OUT_0_1
 Wire Wire Line
-	4800 3200 5400 3200
-Text GLabel 5400 3200 2    70   BiDi ~ 0
+	4800 3200 4850 3200
+Text GLabel 4850 3200 2    70   BiDi ~ 0
 FAULT_OUT_0_0
 Wire Wire Line
@@
 V_CURRENT_3
 $Comp
-L GPA_dortmund-eagle-import:OPA549_KV_11TO-220_11 U11
+L GPA_dortmund-rescue:OPA549_KV_11TO-220_11-GPA_dortmund-eagle-import U11
 U 1 1 6BED38E3
 P 4700 3800
@@
 $EndComp
 $Comp
-L GPA_dortmund-eagle-import:OPA549_KV_11TO-220_11 U12
+L GPA_dortmund-rescue:OPA549_KV_11TO-220_11-GPA_dortmund-eagle-import U12
 U 1 1 6D2AEAA6
 P 7900 3800
@@
 L power:GND #PWR?
 U 1 1 61BC4EC3
-P 8300 6000
+P 8000 6000
 AR Path="/61AB9A1E/61BC4EC3" Ref="#PWR?"  Part="1"
 AR Path="/61AB9CEF/61BC4EC3" Ref="#PWR0123"  Part="1"
-F 0 "#PWR0123" H 8300 5750 50  0001 C CNN
-F 1 "GND" H 8305 5827 50  0000 C CNN
-F 2 "" H 8300 6000 50  0001 C CNN
-F 3 "" H 8300 6000 50  0001 C CNN
-	1    8300 6000
+F 0 "#PWR0123" H 8000 5750 50  0001 C CNN
+F 1 "GND" H 8005 5827 50  0000 C CNN
+F 2 "" H 8000 6000 50  0001 C CNN
+F 3 "" H 8000 6000 50  0001 C CNN
+	1    8000 6000
 	1    0    0    -1
 $EndComp
@@
 $EndComp
 NoConn ~ 6600 4300
+Wire Wire Line
+	8000 3100 8000 3000
+Wire Wire Line
+	8000 3000 8200 3000
+$Comp
+L power:+12V #PWR0146
+U 1 1 61C7D84C
+P 6400 5700
+F 0 "#PWR0146" H 6400 5550 50  0001 C CNN
+F 1 "+12V" H 6415 5873 50  0000 C CNN
+F 2 "" H 6400 5700 50  0001 C CNN
+F 3 "" H 6400 5700 50  0001 C CNN
+	1    6400 5700
+	1    0    0    -1
+$EndComp
 $EndSCHEMATC
