File: GPA PCB files/GPA_dortmund_3.kicad_sch (KiCad schematic)
At the start: 29 parts, among them U10 INA149SOIC8, U101 AAVID_TO220_HEATSINK, U8 OPA549, U9 OPA549, X3 MINI-FIT-JR-045569-NA2

Commit message: converted symbol library to KiCad6 (.kicad_sym)
fixed some pin types to clear ERC and DRC errors/warnings;
added solder jumper to switch from INA149 to LT1990A
fixed layer boundaries (some artifacts from the eagle conversion
Parts:
- added JP2: SolderJumper_2_Open, Jumper:SolderJumper-2_P1.3mm_Open_RoundedPad1.0x1.5mm, symbol Jumper:SolderJumper_2_Open
- U8, U9: symbol GPA_dortmund-rescue:OPA549_KV_11TO-220_11-GPA_dortmund-eagle-import -> GPA_dortmund-eagle-import:OPA549_KV_11TO-220_11
Connections:
- net REF_2.5V: now also JP2.1 (A); no longer U10.5 (REFA)
- new net: JP2.2 (B), U10.5 (REFA)
Changed lines of the file:
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@@
     (stroke (width 0) (type default) (color 0 0 0 0))
   )
-  (wire (pts (xy 160.02 172.72) (xy 142.24 172.72))
+  (wire (pts (xy 160.02 172.72) (xy 156.21 172.72))
     (stroke (width 0) (type default) (color 0 0 0 0))
   )
@@
   )
   (wire (pts (xy 76.2 101.6) (xy 71.12 101.6))
+    (stroke (width 0) (type default) (color 0 0 0 0))
+  )
+  (wire (pts (xy 148.59 172.72) (xy 142.24 172.72))
     (stroke (width 0) (type default) (color 0 0 0 0))
   )
@@
       (effects (font (size 1.27 1.27)) hide)
     )
+    (pin "8")
     (pin "1")
     (pin "2")
@@
     (pin "2")
   )
-  (symbol (lib_id "GPA_dortmund-rescue:OPA549_KV_11TO-220_11-GPA_dortmund-eagle-import") (at 119.38 96.52 0) (unit 1)
+  (symbol (lib_id "GPA_dortmund-eagle-import:OPA549_KV_11TO-220_11") (at 119.38 96.52 0) (unit 1)
     (in_bom yes) (on_board yes)
     (property "Reference" "U8" (id 0) (at 115.57 93.98 0)
@@
     (pin "2")
   )
-  (symbol (lib_id "GPA_dortmund-rescue:OPA549_KV_11TO-220_11-GPA_dortmund-eagle-import") (at 200.66 96.52 0) (mirror y) (unit 1)
+  (symbol (lib_id "GPA_dortmund-eagle-import:OPA549_KV_11TO-220_11") (at 200.66 96.52 0) (mirror y) (unit 1)
     (in_bom yes) (on_board yes)
     (property "Reference" "U9" (id 0) (at 200.66 93.98 0)
@@
       (effects (font (size 1.27 1.27)) hide)
     )
+    (pin "1")
+    (pin "2")
+  )
+  (symbol (lib_id "Jumper:SolderJumper_2_Open") (at 152.4 172.72 0) (unit 1)
+    (in_bom yes) (on_board yes) (fields_autoplaced)
+    (property "Reference" "JP2" (id 0) (at 152.4 166.37 0))
+    (property "Value" "SolderJumper_2_Open" (id 1) (at 152.4 168.91 0))
+    (property "Footprint" "Jumper:SolderJumper-2_P1.3mm_Open_RoundedPad1.0x1.5mm" (id 2) (at 152.4 172.72 0)
+      (effects (font (size 1.27 1.27)) hide)
+    )
+    (property "Datasheet" "~" (id 3) (at 152.4 172.72 0)
+      (effects (font (size 1.27 1.27)) hide)
+    )

Commit message: added 3D models + footprint changes
changed footprints of OPA549T bulk capacitors
Parts:
- C37, C38, C40, C41: footprint GPA_dortmund:C0805 -> Capacitor_SMD:C_1210_3225Metric_Pad1.33x2.70mm_HandSolder
Changed lines of the file:
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@@
       (effects (font (size 1.4986 1.4986)) (justify left bottom))
     )
-    (property "Footprint" "GPA_dortmund:C0805" (id 2) (at 132.08 38.1 0)
+    (property "Footprint" "Capacitor_SMD:C_1210_3225Metric_Pad1.33x2.70mm_HandSolder" (id 2) (at 132.08 38.1 0)
       (effects (font (size 1.27 1.27)) hide)
     )
@@
       (effects (font (size 1.4986 1.4986)) (justify left bottom))
     )
-    (property "Footprint" "GPA_dortmund:C0805" (id 2) (at 121.92 38.1 0)
+    (property "Footprint" "Capacitor_SMD:C_1210_3225Metric_Pad1.33x2.70mm_HandSolder" (id 2) (at 121.92 38.1 0)
       (effects (font (size 1.27 1.27)) hide)
     )
@@
       (effects (font (size 1.4986 1.4986)) (justify left bottom))
     )
-    (property "Footprint" "GPA_dortmund:C0805" (id 2) (at 193.04 38.1 0)
+    (property "Footprint" "Capacitor_SMD:C_1210_3225Metric_Pad1.33x2.70mm_HandSolder" (id 2) (at 193.04 38.1 0)
       (effects (font (size 1.27 1.27)) hide)
     )
@@
       (effects (font (size 1.4986 1.4986)) (justify left bottom))
     )
-    (property "Footprint" "GPA_dortmund:C0805" (id 2) (at 203.2 38.1 0)
-      (effects (font (size 1.27 1.27)) hide)
-    )
+    (property "Footprint" "Capacitor_SMD:C_1210_3225Metric_Pad1.33x2.70mm_HandSolder" (id 2) (at 203.2 38.1 0)
+      (effects (font (size 1.27 1.27)) hide)
+    )
